File: MYiR_24-22_Camface.kicad_sch (KiCad schematic)
At the start: 0 parts

Commit message: Complete schematic and add MIPI CSI differential net class
Co-Authored-By: Claude Sonnet 5.5 <noreply@anthropic.com>
Parts:
- added J1: Conn_01x22_FPC_0.5mm, 0_Custom:FPC_1x22_P0.5mm_Horizontal_BottomContact, symbol 0_Custom:Conn_01x22_FPC_P0.5mm_Horizontal_BottomContact
- added J2: Conn_01x24_FPC, 0_Custom:FPC_1x24_P0.5mm_Horizontal_BottomContact, symbol 0_Custom:Conn_01x24_FPC_P0.5mm_Horizontal_BottomContact
- added JP1: SolderJumper_2_Bridged, PCM_Jumper_AKL:Jumper_P10.16mm_D0.7mm, symbol Jumper:SolderJumper_2_Bridged
- added TP1, TP2: PTH, Connector_Pin:Pin_D1.0mm_L10.0mm, symbol PCM_SparkFun-Connector:TestPoint_PTH
- added TP3, TP4, TP5, TP6, TP7: PTH, Connector_Pin:Pin_D0.7mm_L6.5mm_W1.8mm_FlatFork, symbol PCM_SparkFun-Connector:TestPoint_PTH
Connections:
- new net: J2.23 (Pin_23), JP1.2 (B)
- new net +3.3V: J1.1 (Pin_1), JP1.1 (A), TP1.1
- new net +5V: J2.24 (Pin_24), TP2.1
- new net CKN: J1.15 (Pin_15), J2.7 (Pin_7)
- new net CKP: J1.14 (Pin_14), J2.8 (Pin_8)
- new net D0N: J1.21 (Pin_21), J2.1 (Pin_1)
- new net D0P: J1.20 (Pin_20), J2.2 (Pin_2)
- new net D1N: J1.18 (Pin_18), J2.4 (Pin_4)
- new net D1P: J1.17 (Pin_17), J2.5 (Pin_5)
- new net D2N: J1.12 (Pin_12), J2.10 (Pin_10)
- new net D2P: J1.11 (Pin_11), J2.11 (Pin_11)
- new net D3N: J1.9 (Pin_9), J2.13 (Pin_13)
- new net D3P: J1.8 (Pin_8), J2.14 (Pin_14)
- new net EN: J1.6 (Pin_6), TP6.1
- new net GND: J1.10 (Pin_10), J1.13 (Pin_13), J1.16 (Pin_16), J1.19 (Pin_19), J1.22 (Pin_22), J1.4 (Pin_4), J1.7 (Pin_7), J1.MNT1, J1.MNT2, J2.12 (Pin_12), J2.15 (Pin_15), J2.17 (Pin_17), J2.3 (Pin_3), J2.6 (Pin_6), J2.9 (Pin_9), J2.MNT1, J2.MNT2
- new net GPIO2: J1.5 (Pin_5), TP7.1
- new net MCLK: J2.16 (Pin_16), TP5.1
- new net PWDN: J2.18 (Pin_18), TP3.1
- new net RST: J2.19 (Pin_19), TP4.1
- new net SCL: J1.3 (Pin_3), J2.20 (Pin_20)
- new net SDA: J1.2 (Pin_2), J2.21 (Pin_21)
- no-connect marks 0 -> 1
Other:
- title: (none) -> MYiR 24-22 Camface

Commit message: Add mounting holes, board outline, and component placement
Co-Authored-By: Claude Sonnet 5.5 <noreply@anthropic.com>
Parts:
- removed JP1: SolderJumper_2_Bridged, PCM_Jumper_AKL:Jumper_P10.16mm_D0.7mm, symbol Jumper:SolderJumper_2_Bridged
- added H1, H2: MH, MountingHole:MountingHole_2.7mm_M2.5_DIN965, symbol Mechanical:MountingHole
- added JP3: (no value), PCM_SparkFun-Jumper:Jumper_2_NO, symbol PCM_SparkFun-Jumper:SolderJumper_2_Open
- renumbered TP1 to 3V3, TP2 to 5V, TP6 to EN, TP7 to G2, TP5 to MCK, TP3 to PDN, TP4 to RST
Connections:
- net +3.3V: now also JP3.1 (A)
- net at J2.23 (Pin_23): now also JP3.2 (B)
Changed lines of the file:
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@@
-	(wire
-		(pts
-			(xy 165.1 113.03) (xy 173.99 113.03)
-		)
-		(stroke
-			(width 0)
-			(type default)
-		)
-	)
 	(wire
 		(pts
@@
 	(wire
 		(pts
+			(xy 162.56 113.03) (xy 173.99 113.03)
+		)
+		(stroke
+			(width 0)
+			(type default)
+		)
+	)
+	(wire
+		(pts
 			(xy 107.95 69.85) (xy 107.95 77.47)
 		)
@@
 	(wire
 		(pts
-			(xy 139.7 113.03) (xy 154.94 113.03)
+			(xy 139.7 113.03) (xy 157.48 113.03)
 		)
 		(stroke
@@
 	)
 	(symbol
+		(lib_id "Mechanical:MountingHole")
+		(at 203.2 82.55 0)
+		(unit 1)
+		(body_style 1)
+		(exclude_from_sim no)
+		(in_bom no)
+		(on_board yes)
+		(in_pos_files yes)
+		(dnp no)
+		(fields_autoplaced yes)
+		(property "Reference" "H2"
+			(at 205.74 81.2799 0)
+			(show_name no)
+			(do_not_autoplace no)
+			(effects
+				(font
+					(size 1.27 1.27)
+				)
+				(justify left)
+			)
+		)
+		(property "Value" "MH"
+			(at 205.74 83.8199 0)
+			(show_name no)
+			(do_not_autoplace no)
+			(effects
+				(font
+					(size 1.27 1.27)
+				)
+				(justify left)
+			)
+		)
+		(property "Footprint" "MountingHole:MountingHole_2.7mm_M2.5_DIN965"
+			(at 203.2 82.55 0)
+			(hide yes)
+			(show_name no)
+			(do_not_autoplace no)
+			(effects
+				(font
+					(size 1.27 1.27)
+				)
+			)
+		)
+		(property "Datasheet" ""
+			(at 203.2 82.55 0)
+			(hide yes)
+			(show_name no)
+			(do_not_autoplace no)
+			(effects
+				(font
+					(size 1.27 1.27)
+				)
+			)
+		)
+		(property "Description" "Mounting Hole without connection"
+			(at 203.2 82.55 0)
+			(hide yes)
+			(show_name no)
+			(do_not_autoplace no)
+			(effects
+				(font
+					(size 1.27 1.27)
+				)
+			)
+		)
+		(instances
+			(project "MYiR_24-22_Camface"
+				(path "/537985de-ea24-4fe9-96e4-9dfd7abe623a"
+					(reference "H2")
+					(unit 1)
+				)
+			)
+		)
+	)
+	(symbol
 		(lib_id "PCM_SparkFun-Connector:TestPoint_PTH")
 		(at 160.02 92.71 0)
@@
 		(dnp no)
 		(fields_autoplaced yes)
-		(property "Reference" "TP5"
+		(property "Reference" "MCK"
 			(at 160.02 87.63 0)
 			(show_name no)
@@
 			(project "MYiR_24-22_Camface"
 				(path "/537985de-ea24-4fe9-96e4-9dfd7abe623a"
-					(reference "TP5")
-					(unit 1)
-				)
-			)
-		)
-	)
-	(symbol
-		(lib_id "Jumper:SolderJumper_2_Bridged")
-		(at 160.02 113.03 0)
-		(unit 1)
-		(body_style 1)
-		(exclude_from_sim no)
-		(in_bom no)
-		(on_board yes)
-		(in_pos_files yes)
-		(dnp no)
-		(property "Reference" "JP1"
-			(at 159.766 110.744 0)
-			(show_name no)
-			(do_not_autoplace no)
-			(effects
-				(font
-					(size 1.27 1.27)
-				)
-			)
-		)
-		(property "Value" "SolderJumper_2_Bridged"
-			(at 160.02 109.22 0)
-			(hide yes)
-			(show_name no)
-			(do_not_autoplace no)
-			(effects
-				(font
-					(size 1.27 1.27)
-				)
-			)
-		)
-		(property "Footprint" "PCM_Jumper_AKL:Jumper_P10.16mm_D0.7mm"
-			(at 160.02 113.03 0)
-			(hide yes)
-			(show_name no)
-			(do_not_autoplace no)
-			(effects
-				(font
-					(size 1.27 1.27)
-				)
-			)
-		)
-		(property "Datasheet" ""
-			(at 160.02 119.38 0)
-			(hide yes)
-			(show_name no)
-			(do_not_autoplace no)
-			(effects
-				(font
-					(size 1.27 1.27)
-				)
-			)
-		)
-		(property "Description" "Solder Jumper, 2-pole, closed/bridged"
-			(at 160.02 118.11 0)
-			(hide yes)
-			(show_name no)
-			(do_not_autoplace no)
-			(effects
-				(font
-					(size 1.27 1.27)
-				)
-			)
-		)
-		(pin "1"
-		)
-		(pin "2"
-		)
-		(instances
-			(project "MYiR_24-22_Camface"
-				(path "/537985de-ea24-4fe9-96e4-9dfd7abe623a"
-					(reference "JP1")
+					(reference "MCK")
 					(unit 1)
 				)
@@
 	)
 	(symbol
+		(lib_id "Mechanical:MountingHole")
+		(at 203.2 76.2 0)
+		(unit 1)
+		(body_style 1)
+		(exclude_from_sim no)
+		(in_bom no)
+		(on_board yes)
+		(in_pos_files yes)
+		(dnp no)
+		(fields_autoplaced yes)
+		(property "Reference" "H1"
+			(at 205.74 74.9299 0)
+			(show_name no)
+			(do_not_autoplace no)
+			(effects
+				(font
+					(size 1.27 1.27)
+				)
+				(justify left)
+			)
+		)
+		(property "Value" "MH"
+			(at 205.74 77.4699 0)
+			(show_name no)
+			(do_not_autoplace no)
+			(effects
+				(font
+					(size 1.27 1.27)
+				)
+				(justify left)
+			)
+		)
+		(property "Footprint" "MountingHole:MountingHole_2.7mm_M2.5_DIN965"
+			(at 203.2 76.2 0)
+			(hide yes)
+			(show_name no)
+			(do_not_autoplace no)
+			(effects
+				(font
+					(size 1.27 1.27)
+				)
+			)
+		)
+		(property "Datasheet" ""
+			(at 203.2 76.2 0)
+			(hide yes)
+			(show_name no)
+			(do_not_autoplace no)
+			(effects
+				(font
+					(size 1.27 1.27)
+				)
+			)
+		)
+		(property "Description" "Mounting Hole without connection"
+			(at 203.2 76.2 0)
+			(hide yes)
+			(show_name no)
+			(do_not_autoplace no)
+			(effects
+				(font
+					(size 1.27 1.27)
+				)
+			)
+		)
+		(instances
+			(project "MYiR_24-22_Camface"
+				(path "/537985de-ea24-4fe9-96e4-9dfd7abe623a"
+					(reference "H1")
+					(unit 1)
+				)
+			)
+		)
+	)
+	(symbol
 		(lib_id "PCM_SparkFun-Connector:TestPoint_PTH")
 		(at 139.7 63.5 0)
@@
 		(dnp no)
 		(fields_autoplaced yes)
-		(property "Reference" "TP2"
+		(property "Reference" "5V"
 			(at 139.7 58.42 0)
 			(show_name no)
@@
 			(project "MYiR_24-22_Camface"
 				(path "/537985de-ea24-4fe9-96e4-9dfd7abe623a"
-					(reference "TP2")
+					(reference "5V")
 					(unit 1)
 				)
@@
 		(dnp no)
 		(fields_autoplaced yes)
-		(property "Reference" "TP4"
+		(property "Reference" "RST"
 			(at 147.32 87.63 0)
 			(show_name no)
@@
 			(project "MYiR_24-22_Camface"
 				(path "/537985de-ea24-4fe9-96e4-9dfd7abe623a"
-					(reference "TP4")
+					(reference "RST")
 					(unit 1)
 				)
@@
 		(dnp no)
 		(fields_autoplaced yes)
-		(property "Reference" "TP1"
+		(property "Reference" "3V3"
 			(at 127 58.42 0)
 			(show_name no)
@@
 			(project "MYiR_24-22_Camface"
 				(path "/537985de-ea24-4fe9-96e4-9dfd7abe623a"
-					(reference "TP1")
+					(reference "3V3")
 					(unit 1)
 				)
@@
 		(dnp no)
 		(fields_autoplaced yes)
-		(property "Reference" "TP3"
+		(property "Reference" "PDN"
 			(at 153.67 87.63 0)
 			(show_name no)
@@
 			(project "MYiR_24-22_Camface"
 				(path "/537985de-ea24-4fe9-96e4-9dfd7abe623a"
-					(reference "TP3")
+					(reference "PDN")
+					(unit 1)
+				)
+			)
+		)
+	)
+	(symbol
+		(lib_id "PCM_SparkFun-Jumper:SolderJumper_2_Open")
+		(at 160.02 113.03 0)
+		(unit 1)
+		(body_style 1)
+		(exclude_from_sim no)
+		(in_bom yes)
+		(on_board yes)
+		(in_pos_files yes)
+		(dnp no)
+		(property "Reference" "JP3"
+			(at 160.02 110.744 0)
+			(show_name no)
+			(do_not_autoplace no)
+			(effects
+				(font
+					(size 1.27 1.27)
+				)
+			)
+		)
+		(property "Value" ""
+			(at 160.02 115.57 0)
+			(show_name no)
+			(do_not_autoplace no)
+			(effects
+				(font
+					(size 1.27 1.27)
+				)
+			)
+		)
+		(property "Footprint" "PCM_SparkFun-Jumper:Jumper_2_NO"
+			(at 160.02 116.332 0)
+			(hide yes)
+			(show_name no)
+			(do_not_autoplace no)
+			(effects
+				(font
+					(size 1.27 1.27)
+				)
+			)
+		)
+		(property "Datasheet" ""
+			(at 160.02 119.38 0)
+			(hide yes)
+			(show_name no)
+			(do_not_autoplace no)
+			(effects
+				(font
+					(size 1.27 1.27)
+				)
+			)
+		)
+		(property "Description" "Solder Jumper, 2-pole, open"
+			(at 160.02 121.92 0)
+			(hide yes)
+			(show_name no)
+			(do_not_autoplace no)
+			(effects
+				(font
+					(size 1.27 1.27)
+				)
+			)
+		)
+		(pin "1"
+		)
+		(pin "2"
+		)
+		(instances
+			(project "MYiR_24-22_Camface"
+				(path "/537985de-ea24-4fe9-96e4-9dfd7abe623a"
+					(reference "JP3")
 					(unit 1)
 				)
@@
 		(dnp no)
 		(fields_autoplaced yes)
-		(property "Reference" "TP6"
+		(property "Reference" "EN"
 			(at 88.9 62.23 0)
 			(show_name no)
@@
 			(project "MYiR_24-22_Camface"
 				(path "/537985de-ea24-4fe9-96e4-9dfd7abe623a"
-					(reference "TP6")
+					(reference "EN")
 					(unit 1)
 				)
@@
 		(dnp no)
 		(fields_autoplaced yes)
-		(property "Reference" "TP7"
+		(property "Reference" "G2"
 			(at 95.25 62.23 0)
 			(show_name no)
@@
 			(project "MYiR_24-22_Camface"
 				(path "/537985de-ea24-4fe9-96e4-9dfd7abe623a"
-					(reference "TP7")
+					(reference "G2")
 					(unit 1)
 				)

Commit message: Update schematic
Co-Authored-By: Claude Sonnet 5.5 <noreply@anthropic.com>
Parts:
- renumbered 5V to 5V1, EN to EN1, MCK to MCK1, PDN to PDN1, RST to RST1
Changed lines of the file:
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@@
 		(dnp no)
 		(fields_autoplaced yes)
-		(property "Reference" "MCK"
+		(property "Reference" "MCK1"
 			(at 160.02 87.63 0)
 			(show_name no)
@@
 			(project "MYiR_24-22_Camface"
 				(path "/537985de-ea24-4fe9-96e4-9dfd7abe623a"
-					(reference "MCK")
+					(reference "MCK1")
 					(unit 1)
 				)
@@
 		(dnp no)
 		(fields_autoplaced yes)
-		(property "Reference" "5V"
+		(property "Reference" "5V1"
 			(at 139.7 58.42 0)
 			(show_name no)
@@
 			(project "MYiR_24-22_Camface"
 				(path "/537985de-ea24-4fe9-96e4-9dfd7abe623a"
-					(reference "5V")
+					(reference "5V1")
 					(unit 1)
 				)
@@
 		(dnp no)
 		(fields_autoplaced yes)
-		(property "Reference" "RST"
+		(property "Reference" "RST1"
 			(at 147.32 87.63 0)
 			(show_name no)
@@
 			(project "MYiR_24-22_Camface"
 				(path "/537985de-ea24-4fe9-96e4-9dfd7abe623a"
-					(reference "RST")
+					(reference "RST1")
 					(unit 1)
 				)
@@
 		(dnp no)
 		(fields_autoplaced yes)
-		(property "Reference" "PDN"
+		(property "Reference" "PDN1"
 			(at 153.67 87.63 0)
 			(show_name no)
@@
 			(project "MYiR_24-22_Camface"
 				(path "/537985de-ea24-4fe9-96e4-9dfd7abe623a"
-					(reference "PDN")
+					(reference "PDN1")
 					(unit 1)
 				)
@@
 		(dnp no)
 		(fields_autoplaced yes)
-		(property "Reference" "EN"
+		(property "Reference" "EN1"
 			(at 88.9 62.23 0)
 			(show_name no)
@@
 			(project "MYiR_24-22_Camface"
 				(path "/537985de-ea24-4fe9-96e4-9dfd7abe623a"
-					(reference "EN")
-					(unit 1)
-				)
+					(reference "EN1")
+					(unit 1)
+				)
